File: Hardware/Qwiic GPS-RTK - ublox NEO-M8P.brd (EAGLE design)
At the start: 40.6 x 33 mm, 101 parts, among them J13 U.FL, J3 PTH, U1 NEO-M8P, U2 3.3V

Commit message: Adding examples
Parts:
- removed JP11: SPI, SparkFun-Connectors:1X06_NO_SILK
- removed U$42, U$45: (no value), Labels:MISO
- removed U$46, U$47: (no value), Labels:MOSI
- removed U$48, U$49: (no value), Labels:SCK-[)
- removed U$50, U$59: (no value), Labels:CS#-[>
- added J1: (no value), SparkFun-Connectors:1X07_NO_SILK
- added U$19, U$20: (no value), Labels:5V
- added U$23, U$24: (no value), Labels:CS#-<]
- added U$26, U$33: (no value), Labels:MISO-(]-04
- added U$34, U$37: (no value), Labels:MOSI-(]-04
- added U$38, U$41: (no value), Labels:SCK-(]-04
- D1: value BLUE -> Yellow
- JP15: value SPI -> (none)
- moved C6 22.3 mm to (33.7, 16.1), turned to 270 degrees
- moved C5 20.0 mm to (15.2, 6.99)
- moved R15 19.8 mm to (16.5, 29.2), turned to 270 degrees
- moved U2 18.1 mm to (31.0, 16.1), turned to 90 degrees
- moved C4 14.4 mm to (28.3, 16.1), turned to 90 degrees
- moved U$62 5.45 mm to (19.1, 26.5), turned to 90 degrees
- moved U$63 5.45 mm to (19.1, 26.5), turned to 90 degrees
- moved U$55 5.27 mm to (29.6, 24.9)
- moved U$60 4.70 mm to (24.1, 26.7), turned to 90 degrees
- moved U$61 4.70 mm to (24.1, 26.7), turned to 90 degrees
- moved C1 3.05 mm to (32.8, 18.7), turned to 0 degrees
- moved J13 1.65 mm to (31.4, 22.4)
- moved R14 1.37 mm to (29.5, 18.7), turned to 180 degrees
- moved FB1 1.28 mm to (28.6, 21.1)
Connections:
- net 3.3V: now also J1.3; no longer JP11.2
- net 5V: now also J1.2
- net GND: now also J1.1; no longer JP11.1
- net RXI/MOSI: now also J1.5; no longer JP11.4
- net SCL/SCK: now also J1.7; no longer JP11.6
- net SDA/!CS: now also J1.4; no longer JP11.3
- net TXO/MISO: now also J1.6; no longer JP11.5
Routing:
- net 5V: track 21.3 -> 53.6 mm
- net N$11: track 25.6 -> 55.6 mm
- net N$12: track 24.4 -> 52.2 mm
- net PPS: track 29.3 -> 38.9 mm, vias 3 -> 5
- net INT: track 15.5 -> 24.0 mm
- net FENCE_STAT: track 56.6 -> 51.4 mm, vias 2 -> 3
- net RTK_STAT: track 49.4 -> 53.9 mm, vias 2 -> 4
- net !RESET: track 30.5 -> 28.0 mm
- net SDA/!CS: track 85.4 -> 87.3 mm, vias 2 -> 4
- net !SAFE: track 16.3 -> 18.0 mm, vias 2 -> 1
- net N$13: track 2.03 -> 3.45 mm
- net TXO/MISO: track 37.1 -> 35.8 mm
- net D_SEL: track 2.67 -> 3.95 mm
- net ANT_VCC: track 3.27 -> 4.53 mm
- net GND: track 6.85 -> 5.71 mm, vias 20 -> 161
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Other:
- board text added: "x02"
- board text removed: "x01"

Commit message: Modifications for reds.
Parts:
- removed U$2: SPARKX-LOGO4, SparkX:SPARKX-MEDIUM
- added LOGO2: SFE_LOGO_NAME_FLAME.1_INCH, SparkFun-Aesthetics:SFE_LOGO_NAME_FLAME_.1
- U$26: device Labels:MISO-(]-04 -> buzzard_labels (36):RX#MOSI2
- U$31: value SPARKX-LOGO3 -> (none); device SparkX:SPARKX-SMALL -> buzzard_labels (36):RX#MOSI3
- U$33: device Labels:MISO-(]-04 -> SparkFun-Aesthetics:SFE_LOGO_FLAME_.1
- U$34: device Labels:MOSI-(]-04 -> buzzard_labels (36):TX#MISO0
- U$37: device Labels:MOSI-(]-04 -> buzzard_labels (36):TX#MISO1
- moved U$31 8.26 mm to (29.2, 24.3), flipped to the bottom
- moved U$33 7.03 mm to (38.4, 23.6), flipped to the top
- moved U$55 6.38 mm to (34.2, 20.4), turned to 90 degrees
- moved U$37 3.18 mm to (31.8, 24.1)
- moved U$34 2.74 mm to (31.8, 25.0)
- moved U$26 2.69 mm to (29.2, 25.1)
- moved U$43 0.25 mm to (14.0, 1.65)
- moved U$44 0.25 mm to (14.0, 1.65)
- moved U$14 0.13 mm to (8.89, 1.78)
- moved U$17 0.13 mm to (8.89, 1.78)
- renumbered JP51 to JP5
Other:
- board text added: "v10"
- board text removed: "x02"
