File: Hardware/Production/Qwiic GPS-RTK - ublox NEO-M8P-Panel - Single.brd (EAGLE design)
At the start: 40.6 x 33 mm, 106 parts, among them J13 U.FL, J3 PTH, U1 NEO-M8P, U2 3.3V

Commit message: Adding examples
Parts:
- removed FRAME1: FRAME-LETTER, SparkFun-Aesthetics:CREATIVE_COMMONS
- removed JP11: SPI, SparkFun-Connectors:1X06_NO_SILK
- removed JP12, JP14: (no value), SparkFun-Jumpers:SMT-JUMPER_2_NC_TRACE_SILK
- removed JP13: (no value), SparkFun-Jumpers:SMT-JUMPER_2_NO_SILK
- removed JP6, JP7, JP8: FIDUCIALUFIDUCIAL, SparkFun:MICRO-FIDUCIAL
- removed U$42, U$45: (no value), Labels:MISO
- removed U$46, U$47: (no value), Labels:MOSI
- removed U$48, U$49: (no value), Labels:SCK-[)
- removed U$50, U$59: (no value), Labels:CS#-[>
- removed U$51: (no value), buzzard_labels (32):GPS1
- added E$1, E$2, E$3, E$4: (no value), SparkFun-Aesthetics:FIDUCIAL-1X2
- added E$5, E$6: (no value), SparkFun-Retired:FIDUCIAL-1.5X3
- added J1: (no value), SparkFun-Connectors:1X07_NO_SILK
- added JP21, JP61, JP71, JP81: FIDUCIALUFIDUCIAL, SparkFun:MICRO-FIDUCIAL
- added JP31, JP41: STAND-OFF, SparkFun:STAND-OFF
- added U$34: (no value), Labels:MOSI-(]-04
- added U$38, U$41: (no value), Labels:SCK-(]-04
- added U$53: (no value), buzzard_labels (7):NEO#M8P3
- added U$54: (no value), buzzard_labels (8):GPS#RTK1
- added U$55: (no value), buzzard_labels (9):ANT0
- JP2: value FIDUCIALUFIDUCIAL -> (none); device SparkFun:MICRO-FIDUCIAL -> SparkFun-Jumpers:SMT-JUMPER_2_NC_TRACE_SILK
- JP3: value STAND-OFF -> (none); device SparkFun:STAND-OFF -> SparkFun-Jumpers:SMT-JUMPER_2_NC_TRACE_SILK
- JP4: value STAND-OFF -> (none); device SparkFun:STAND-OFF -> SparkFun-Jumpers:SMT-JUMPER_2_NO_SILK
- R10, R9: value 33 -> 27
- U$18: device buzzard_labels (2):GPS#RTK0 -> Labels:PWR-()-03
- U$19: device buzzard_labels (3):GPS#RTK1 -> Labels:5V
- U$20: device buzzard_labels (2):NEO#M8P2 -> Labels:5V
- U$23: device buzzard_labels (2):NEO#M8P3 -> Labels:CS#-<]
- U$24: device buzzard_labels (3):NEO#M8P2 -> Labels:CS#-<]
- U$26: device buzzard_labels (5):U#BLOX3 -> Labels:MISO-(]-04
- U$31: value SPARKX-LOGO4 -> SPARKX-LOGO3; device SparkX:SPARKX-MEDIUM -> SparkX:SPARKX-SMALL
- U$33: device buzzard_labels (5):JP43 -> Labels:MISO-(]-04
- U$37: device buzzard_labels (30):3V30 -> Labels:MOSI-(]-04
- moved U$30 71.1 mm to (4.19, 8.76)
- moved LOGO1 48.7 mm to (2.54, 26.7)
- moved JP3 40.9 mm to (35.6, 6.35), flipped to the bottom
- moved U$20 35.1 mm to (21.6, 27.7), flipped to the bottom, turned to 90 degrees
- moved U$2 31.8 mm to (20.3, 21.6)
- moved U$22 29.9 mm to (25.3, 18.2)
- moved U$23 29.9 mm to (26.7, 27.9), turned to 90 degrees
- moved U$33 29.5 mm to (31.8, 26.0), flipped to the bottom, turned to 90 degrees
- moved U$19 28.9 mm to (21.6, 27.7), turned to 90 degrees
- moved U$24 27.9 mm to (26.7, 27.9), flipped to the bottom, turned to 90 degrees
- moved C6 22.3 mm to (33.7, 16.1), turned to 270 degrees
- moved JP4 22.2 mm to (29.2, 10.2), flipped to the bottom
- moved U$18 20.4 mm to (28.8, 12.7)
- moved C5 20.0 mm to (15.2, 6.99)
- moved R15 19.8 mm to (16.5, 29.2), turned to 270 degrees
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- renumbered JP10 to JP101, JP5 to JP51, JP9 to JP91
Connections:
- net 3.3V: now also J1.3; no longer JP11.2
- net 5V: now also J1.2
- net D_SEL: now also JP4.2; no longer JP13.2
- net FENCE_STAT: now also JP3.2; no longer JP14.2
- net GND: now also J1.1, JP4.1; no longer JP11.1, JP13.1
- net N$3: now also JP2.1; no longer JP12.1
- net N$9: now also JP3.1; no longer JP14.1
- net RTK_STAT: now also JP2.2; no longer JP12.2
- net RXI/MOSI: now also J1.5; no longer JP11.4
- net SCL/SCK: now also J1.7; no longer JP11.6
- net SDA/!CS: now also J1.4; no longer JP11.3
- net TXO/MISO: now also J1.6; no longer JP11.5
Routing:
- net 5V: track 21.5 -> 53.6 mm
- net N$11: track 25.6 -> 55.8 mm
- net N$12: track 24.4 -> 52.4 mm
- net INT: track 15.5 -> 24.0 mm
- net FENCE_STAT: track 56.6 -> 51.4 mm, vias 2 -> 3
- net RTK_STAT: track 49.4 -> 53.9 mm, vias 2 -> 4
- net !RESET: track 30.5 -> 27.6 mm
- net SDA/!CS: track 85.4 -> 87.4 mm, vias 2 -> 4
- net !SAFE: track 16.3 -> 18.2 mm, vias 2 -> 1
- net GND: track 6.37 -> 8.19 mm, vias 20 -> 161
- net N$13: track 2.03 -> 3.45 mm
- net D_SEL: track 2.67 -> 3.95 mm
- net PPS: track 29.3 -> 30.6 mm, vias 3 -> 2
- net ANT_VCC: track 3.27 -> 4.53 mm
- net TXO/MISO: track 37.1 -> 35.9 mm
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Other:
- board size 40.6 x 33 mm -> 95.5 x 94.2 mm
- board text added: "Route Out"
- board text added: "v-score"
- board text added: "x02"
- board text removed: "Measurements in inches"
- board text removed: "x01"
