File: Hardware/Jig/Qwiic GPS-RTK - ublox NEO-M8P-BottomJig.sch (EAGLE design)
At the start: 19 parts, among them U1 FLYING_JALAPENO, U2 74LVC4066

Commit message: Updating test jig to one button, add ground plane.
Parts:
- removed BUTTON1: CAPSENSE_BUTTON_PAD_ONLY, Testing:CAPSENSE_BUTTON_PAD_ONLY
- removed H2, H4: STAND-OFF, SparkFun-Hardware:STAND-OFF
- added FRAME1: FRAME-LETTER, SparkFun-Aesthetics:FRAME-LETTER
- added J3: PTH, SparkX:I2C_STANDARD_NO_SILK
- added JP101, JP31, JP41, JP91: STAND-OFF, SparkFun:STAND-OFF
- added LOGO1: OSHW-LOGOMINI, SparkFun-Aesthetics:OSHW-LOGOMINI
- added LOGO2: SFE_LOGO_NAME_FLAME.1_INCH, SparkFun-Aesthetics:SFE_LOGO_NAME_FLAME.1_INCH
Connections:
- net N$18 renamed BUTTON2
- removed net 3V3_OUT_FROM_GPS: J1.3, U1.A0
- removed net N$19: BUTTON1.CAPSENSE, U1.CAP_PAD1
- new net 3.3V: J1.3, J3.VCC
- new net 5V: J1.2
- new net JALAPENO_SPI_EN: U1.24
- new net J_25: U1.25
- new net J_26: U1.26
- new net J_27: U1.27
- new net J_28: U1.28
- new net J_A0: U1.A0
- new net TARGET_RX: J_SCL1.2, U2.3Z
- new net TARGET_SCL: J_SCL.2, U2.2Z
- new net TARGET_SDA: J_SCL2.2, U2.1Z
- new net TARGET_TX: J_SDA.2, U2.4Z
- net !RESET: no longer U1.27
- net 5V_POWER: no longer J1.2
- net FENCE_STAT: no longer U1.24
- net GND: now also J3.GND
- net INT: no longer U1.28
- net PPS: no longer U1.26
- net RTK_STAT: no longer U1.25
- net RXI/MOSI: no longer J_SCL1.2, U2.3Z
- net SCL/SCK: now also J3.SCL; no longer J_SCL.2, U2.2Z
- net SDA/!CS: now also J3.SDA; no longer J_SCL2.2, U2.1Z
- net TXO/MISO: no longer J_SDA.2, U2.4Z
Other:
- note added: "7-bit unshifted I2C address: 0x42"
- note added: "CI160808-33NJ"
- note added: "Close jumper to enable SPI"
- note added: "Cut jumper to disable LED"
- note added: "Cut jumper to remove I2C pullups from bus"
- note added: "RTC Backup"
- note added: "Stat LEDs"
- note added: "Ublox NEO-M8P"
- note added: "V10"
- moved on the sheet: J1, JP15
